File: KiCad/M2MRover_Power.sch (KiCad schematic (older format))
At the start: 8 parts, among them SW1 SW_SPST, U3 LD1117V50, U4 LD1117V33

Commit message: Route the PCB
Parts:
- BT1, SW1: footprint (none) -> Connector_PinHeader_2.54mm:PinHeader_1x02_P2.54mm_Vertical
Changed lines of the file:
@@
 F 0 "BT1" H 2708 2346 50  0000 L CNN
 F 1 "Battery" H 2708 2255 50  0000 L CNN
-F 2 "" V 2600 2360 50  0001 C CNN
+F 2 "Connector_PinHeader_2.54mm:PinHeader_1x02_P2.54mm_Vertical" V 2600 2360 50  0001 C CNN
 F 3 "~" V 2600 2360 50  0001 C CNN
 	1    2600 2300
@@
 F 0 "SW1" H 2300 2185 50  0000 C CNN
 F 1 "SW_SPST" H 2300 2094 50  0000 C CNN
-F 2 "" H 2300 1950 50  0001 C CNN
+F 2 "Connector_PinHeader_2.54mm:PinHeader_1x02_P2.54mm_Vertical" H 2300 1950 50  0001 C CNN
 F 3 "~" H 2300 1950 50  0001 C CNN
 	1    2300 1950
